File: KiCad/remote control adapter.kicad_sch (KiCad schematic)
At the start: 28 parts, among them J1 0, J2 0, Q1 DTA124EUA

Commit message: Add files via upload
Updated a few capacitor values
Parts:
- C11, C12: value 2.2n -> 1n
- C39: value 0.47 -> 1n
